Commit message: Add moveit config package for scara

File: docker/irb910sc-planner/abb_irb910sc_support/urdf/irb910sc_3_065.urdf (robot description, URDF)
Before this commit: robot irb910, 6 links, 5 joints
Links:
- added link flange
- added link tool0
Joints:
- added joint flange: type fixed, parent link4, child flange, origin xyz=0.0 0.0 0.0 rpy=0.0 -0.0 0.0, axis 0.0 0.0 1.0
- added joint link_6-tool0: type fixed, parent flange, child tool0, origin xyz=0.0 0.0 0.0 rpy=0.0 -0.0 0.0, axis 0.0 0.0 1.0

Commit message: Fix urdf

File: docker/irb910sc-planner/abb_irb910sc_support/urdf/irb910sc_3_065.urdf (robot description, URDF)
Before this commit: robot irb910, 8 links, 7 joints
Joints:
- removed joint flange
- removed joint link_6-tool0
- added joint flange-tool0: type fixed, parent flange, child tool0, origin xyz=0.0 0.0 0.0 rpy=0.0 -0.0 0.0
- added joint link_4-flange: type fixed, parent link4, child flange, origin xyz=0.0 0.0 0.0 rpy=0.0 -0.0 0.0
- joint base_link-base: axis 0.0 0.0 1.0 -> (none)
- joint joint3: limit lower=-0.18 effort=0.0 velocity=0.0 -> lower=-0.18 upper=0.0 effort=0.0 velocity=0.0
